Commit message: added moveit and controllers

File: robot_description/maciv2.urdf.xacro (robot description, xacro)
@@ -2,5 +2,6 @@
 <robot xmlns:xacro="http://www.ros.org/wiki/xacro" name="maciv2">
     <!-- Robot stuff goes here -->
-    <xacro:include filename="$(find ur_description)/urdf/ur_macro.xacro"/>
+    <xacro:include filename="$(find krytn)/robot_description/magni/inertial.xacro" />
+    <xacro:include filename="$(find ur_description)/urdf/ur_macro.xacro" />
     <xacro:arg name="ur_type" default="ur5e"/>
     <xacro:ur_robot name="ur5" tf_prefix="ur5_" parent="world" joint_limits_parameters_file="$(find ur_description)/config/$(arg ur_type)/joint_limits.yaml" kinematics_parameters_file="$(find ur_description)/config/$(arg ur_type)/default_kinematics.yaml" physical_parameters_file="$(find ur_description)/config/$(arg ur_type)/physical_parameters.yaml" visual_parameters_file="$(find ur_description)/config/$(arg ur_type)/visual_parameters.yaml" sim_ignition="true" initial_positions="${dict(shoulder_pan_joint=-0.15,shoulder_lift_joint=0,elbow_joint=0.0,wrist_1_joint=0,wrist_2_joint=0.0,wrist_3_joint=0.0)}">
@@ -8,3 +9,64 @@
     </xacro:ur_robot>
     <link name="world" />
+    <joint name="gripper_joint" type="fixed">
+        <origin xyz="0.0 0.0 0.0" rpy="0.0 -${pi/2} 0.0" />
+        <parent link="ur5_tool0" />
+        <child link="gripper_base_link" />
+    </joint>
+    <link name="gripper_base_link">
+        <visual>
+            <!--gripper_base-->
+            <geometry>
+                <mesh filename="file://$(find maciv2)/robot_description/meshes/gripper2_gripper_base.dae"/>
+            </geometry>
+        </visual>
+        <collision>
+            <!--gripper_base-->
+            <geometry>
+                <mesh filename="file://$(find maciv2)/robot_description/meshes/gripper2_gripper_base.dae"/>
+            </geometry>
+        </collision>
+    </link>
+    <link name="finger_link">
+        <visual>
+            <!--finger-->
+            <origin rpy="0.0 -0.0 0.0" xyz="0.0 0.0 0.0"/>
+            <geometry>
+                <mesh filename="file://$(find maciv2)/robot_description/meshes/gripper2_finger.dae"/>
+            </geometry>
+        </visual>
+        <collision>
+            <!--finger-->
+            <origin rpy="0.0 -0.0 0.0" xyz="0.0 0.0 0.0"/>
+            <geometry>
+                <mesh filename="file://$(find maciv2)/robot_description/meshes/gripper2_finger.dae"/>
+            </geometry>
+        </collision>
+        <xacro:box_inertial x="0.03" y="0.03" z="0.1" mass="1" />
+    </link>
+    <joint name="finger_joint" type="prismatic">
+        <parent link="gripper_base_link"/>
+        <child link="finger_link"/>
+        <origin rpy="0.0 0.0 0.0" xyz="0.07 -0.002 0.0578"/>
+        <axis xyz="0 0 1"/>
+        <limit effort="1000.0" lower="-0.08" upper="0.0" velocity="10.0"/>
+    </joint>
+    <!-- Configure Control of Joints -->
+    <ros2_control name="maciv2" type="system">
+        <hardware>
+            <plugin>ign_ros2_control/IgnitionSystem</plugin>
+        </hardware>
+        <joint name="finger_joint">
+            <command_interface name="position"/>
+            <state_interface name="position">
+                <param name="initial_value">0.0</param>
+            </state_interface>
+            <state_interface name="velocity"/>
+        </joint>
+    </ros2_control>
+    <gazebo>
+        <plugin filename="ign_ros2_control-system" name="ign_ros2_control::IgnitionROS2ControlPlugin">
+            <parameters>$(find maciv2)/config/ros2_controllers.yaml</parameters>
+        </plugin>
+    </gazebo>
 </robot>

Commit message: added gazebo sensors to maci urdf xacro file, modified the realsense topics in launch files and urdf and finally added the folder in the setup.py

File: robot_description/maciv2.urdf.xacro (robot description, xacro)
@@ -9,4 +9,9 @@
     </xacro:ur_robot>
     <link name="world" />
+    <xacro:include filename="$(find realsense2_description)/urdf/_d435i.urdf.xacro" />
+    <!-- Including realsense description from external package -->
+    <xacro:sensor_d435i parent="ur5_base_link" name="sensor_d435i" use_nominal_extrinsics="True">
+        <origin xyz="-1 -1 0.5" rpy="0 0 ${pi/4}"/>
+    </xacro:sensor_d435i>
     <joint name="gripper_joint" type="fixed">
         <origin xyz="0.0 0.0 0.0" rpy="0.0 -${pi/2} 0.0" />
@@ -69,4 +74,38 @@
             <parameters>$(find maciv2)/config/ros2_controllers.yaml</parameters>
         </plugin>
+        <plugin filename="ignition-gazebo-sensors-system" name="ignition::gazebo::systems::Sensors">
+            <render_engine>ogre2</render_engine>
+        </plugin>
+    </gazebo>
+    <!-- Add sensor tags to Realsense links -->
+    <gazebo reference="sensor_d435i_link">
+        <sensor name="realsense_d435" type="rgbd_camera">
+            <topic>realsense</topic>
+            <ignition_frame_id>sensor_d435i_link</ignition_frame_id>
+            <update_rate>5</update_rate>
+            <camera name="camera">
+                <horizontal_fov>1.5</horizontal_fov>
+                <image>
+                    <width>320</width>
+                    <height>240</height>
+                    <format>R8G8B8</format>
+                </image>
+                <clip>
+                    <near>0.01</near>
+                    <far>10</far>
+                </clip>
+                <depth_camera>
+                    <clip>
+                        <near>0.1</near>
+                        <far>10</far>
+                    </clip>
+                </depth_camera>
+                <noise>
+                    <type>gaussian</type>
+                    <mean>0</mean>
+                    <stddev>0.007</stddev>
+                </noise>
+            </camera>
+        </sensor>
     </gazebo>
 </robot>
